File: Doc/Schematic/6502 Sandbox/6502 Sandbox.kicad_sch (KiCad schematic)
At the start: 25 parts, among them U1 W65C02SxP, U2 W65C22NxP, U5 74HC00

Commit message: feat: First version complete
Parts:
- added U? (x4): 74HC00, symbol 74xx:74HC00
- added U?: 28C256, symbol Memory_EEPROM:28C256
- added U?: KM62256CLP, Package_DIP:DIP-28_W15.24mm, symbol Memory_RAM:KM62256CLP
Connections:
- net A0: now also U?.10 (A0), U?.10 (A0)
- net A1: now also U?.9 (A1), U?.9 (A1)
- net A10: now also U?.21 (A10), U?.21 (A10)
- net A11: now also U?.23 (A11), U?.23 (A11)
- net A12: now also U?.2 (A12)
- net A13: now also U?.10
- net A14: now also U?.2, U?.22 (~{OE})
- net A15: now also U?.1
- net A2: now also U?.8 (A2), U?.8 (A2)
- net A3: now also U?.7 (A3), U?.7 (A3)
- net A4: now also U?.6 (A4), U?.6 (A4)
- net A5: now also U?.5 (A5), U?.5 (A5)
- net A6: now also U?.4 (A6), U?.4 (A6)
- net A7: now also U?.3 (A7), U?.3 (A7)
- net A8: now also U?.25 (A8), U?.25 (A8)
- net A9: now also U?.24 (A9), U?.24 (A9)
- net D0: now also U?.11 (D0), U?.11 (Q0)
- net D1: now also U?.12 (D1), U?.12 (Q1)
- net D2: now also U?.13 (D2), U?.13 (Q2)
- net D3: now also U?.15 (D3), U?.15 (Q3)
- net D4: now also U?.16 (D4), U?.16 (Q4)
- net D5: now also U?.17 (D5), U?.17 (Q5)
- net D6: now also U?.18 (D6), U?.18 (Q6)
- net D7: now also U?.19 (D7), U?.19 (Q7)
- net GND: now also U?.14 (GND), U?.14 (GND), U?.20 (~{CS}), U?.20 (~{CS})
- net VDD: now also U?.27 (~{WE}), U?.28 (VCC), U?.28 (VCC)
- net at U1.34 (R/~{W}), U2.22 (R/~{W}): now also U?.27 (~{WE})
- new net: U?.22 (~{OE}), U?.8
- new net: U?.6, U?.9
- new net: U?.3, U?.4, U?.5
Other:
- note added: "2022/02/12"
- note added: "EEPROM $E000 --> $FFFF"
- note added: "LCD_RS .equ $80 ;PORTA_7 LCD_RWB .equ $40 ;PORTA_6 LCD_E .equ $20 ;PORTA_5"
- note added: "RAM $0000 --> $1FFF"
- note added: "VIA $6000"
- note removed: ";LCD LCD_RS .equ $80 ;PORTA_7 LCD_RWB .equ $40 ;PORTA_6 LCD_E .equ $20 ;PORTA_5"
- note removed: "VIA .equ $6000"
- moved on the sheet: U5D
